Commit message: replace _ with  in ecm.urdf.xacro

File: dvrk_model/model/ECM.urdf.xacro (robot description, xacro)
@@ -1,9 +1,9 @@
 <?xml version="1.0" ?>
-<robot name="ecm" xmlns:xacro="http://www.ros.org/wiki/xacro">
+<robot name="dvrk_ecm" xmlns:xacro="http://www.ros.org/wiki/xacro">
   <!-- Macros -->
   <xacro:include filename="$(find dvrk_model)/model/ecm.urdf.xacro"/>
   <link name="world"/>
   <xacro:ecm
-      prefix="ecm"
+      prefix="$(arg prefix)"
       parent_link="world"
       xyz="0.0 0.0 0.0" rpy="0.0 0.0 0.0"/>

File: dvrk_model/model/ecm.urdf.xacro (robot description, xacro)
@@ -8,15 +8,15 @@
     <joint name="setup_fixed_joint" type="fixed">
       <parent link="${parent_link}"/>
-      <child link="${prefix}_setup_base_link"/>
+      <child link="${prefix}setup_base_link"/>
       <origin rpy="${rpy}" xyz="${xyz}"/>
     </joint>
-    <link name="${prefix}_setup_base_link"/>
+    <link name="${prefix}setup_base_link"/>
     <joint name="setup_tip_joint" type="fixed">
-      <parent link="${prefix}_setup_base_link"/>
-      <child link="${prefix}_setup_link"/>
+      <parent link="${prefix}setup_base_link"/>
+      <child link="${prefix}setup_link"/>
       <origin rpy="-0.87046370379 0 -${PI/2}" xyz="0.91324 -0.02111 0.03166"/>
       <axis xyz="0 0 1"/>
     </joint>
-    <link name="${prefix}_setup_link">
+    <link name="${prefix}setup_link">
       <visual>
         <origin rpy="0 0 0" xyz="0 0 0"/>
@@ -35,13 +35,13 @@
     <!-- Joint 0: Fixed to Setup Joint-->
     <joint name="fixed_joint" type="fixed">
-      <parent link="${prefix}_setup_link"/>
-      <child link="${prefix}_base_link"/>
+      <parent link="${prefix}setup_link"/>
+      <child link="${prefix}base_link"/>
       <origin rpy="0 0 0" xyz="0 0.603 0"/>
     </joint>
-    <link name="${prefix}_base_link"/>
+    <link name="${prefix}base_link"/>
     <!-- Joint 1: Outer Yaw -->
     <joint name="outer_yaw" type="revolute">
-      <parent link="${prefix}_base_link"/>
-      <child link="${prefix}_yaw_link"/>
+      <parent link="${prefix}base_link"/>
+      <child link="${prefix}yaw_link"/>
       <origin rpy="0 -${PI/2} ${PI/2}" xyz="0 0 0"/>
       <axis xyz="0 0 1"/>
@@ -51,5 +51,5 @@
       <joint_properties damping="1.0" friction="0.0"/>
     </joint>
-    <link name="${prefix}_yaw_link">
+    <link name="${prefix}yaw_link">
       <visual>
         <origin rpy="0 0 -${PI/2}" xyz="0.0 0 0.603"/>
@@ -68,6 +68,6 @@
     <!-- Joint 2: Pitch -->
     <joint name="outer_pitch" type="revolute">
-      <parent link="${prefix}_yaw_link"/>
-      <child link="${prefix}_pitch_link"/>
+      <parent link="${prefix}yaw_link"/>
+      <child link="${prefix}pitch_link"/>
       <origin rpy="-${PI/2} -${PI/2} 0" xyz="0 0 0"/>
       <axis xyz="0 0 1"/>
@@ -75,8 +75,8 @@
       <joint_properties damping="1.0" friction="0.0"/>
     </joint>
-    <link name="${prefix}_pitch_link"/>
+    <link name="${prefix}pitch_link"/>
     <joint name="outer_pitch_0" type="continuous">
-      <parent link="${prefix}_yaw_link"/>
-      <child link="${prefix}_pitch_link_1"/>
+      <parent link="${prefix}yaw_link"/>
+      <child link="${prefix}pitch_link_1"/>
       <origin rpy="-${PI/2} -${PI/2} 0" xyz="0 0 0.378"/>
       <axis xyz="0 0 1"/>
@@ -84,5 +84,5 @@
       <mimic joint="outer_pitch" multiplier="1"/>
     </joint>
-    <link name="${prefix}_pitch_link_1">
+    <link name="${prefix}pitch_link_1">
       <visual>
         <origin rpy="${PI} 0 ${PI*78.5/180}" xyz="0.0 0 0.0"/>
@@ -104,6 +104,6 @@
     </link>
     <joint name="outer_pitch_1" type="continuous">
-      <parent link="${prefix}_pitch_link_1"/>
-      <child link="${prefix}_pitch_link_2"/>
+      <parent link="${prefix}pitch_link_1"/>
+      <child link="${prefix}pitch_link_2"/>
       <origin rpy="0 0 0" xyz="0.0558629 0.274575 0"/>
       <axis xyz="0 0 1"/>
@@ -111,5 +111,5 @@
       <mimic joint="outer_pitch" multiplier="-1"/>
     </joint>
-    <link name="${prefix}_pitch_link_2">
+    <link name="${prefix}pitch_link_2">
       <visual>
         <origin rpy="0 0 0" xyz="0.0 0 -0.0225"/>
@@ -131,6 +131,6 @@
     </link>
     <joint name="outer_pitch_2" type="continuous">
-      <parent link="${prefix}_pitch_link_2"/>
-      <child link="${prefix}_pitch_link_3"/>
+      <parent link="${prefix}pitch_link_2"/>
+      <child link="${prefix}pitch_link_3"/>
       <origin rpy="0 0 0" xyz="-0.340 0 0"/>
       <axis xyz="0 0 1"/>
@@ -138,5 +138,5 @@
       <mimic joint="outer_pitch" multiplier="1"/>
     </joint>
-    <link name="${prefix}_pitch_link_3">
+    <link name="${prefix}pitch_link_3">
       <visual>
         <origin rpy="0 0 -${PI/2}" xyz="0.0 0 0.025"/>
@@ -159,6 +159,6 @@
     <!-- Joint 3: Insertion -->
     <joint name="insertion" type="prismatic">
-      <parent link="${prefix}_pitch_link"/>
-      <child link="${prefix}_insertion_link"/>
+      <parent link="${prefix}pitch_link"/>
+      <child link="${prefix}insertion_link"/>
       <origin rpy="${PI/2} 0 0" xyz="0 0.3822 0"/>
       <axis xyz="0 0 1"/>
@@ -166,5 +166,5 @@
       <limit effort="100.0" lower="0" upper="0.235" velocity="10"/>
     </joint>
-    <link name="${prefix}_insertion_link">
+    <link name="${prefix}insertion_link">
       <visual>
         <origin rpy="0 0 -${PI/2}" xyz="0.0 0 -0.015"/>
@@ -183,6 +183,6 @@
     <!-- Joint 4: Roll -->
     <joint name="outer_roll" type="revolute">
-      <parent link="${prefix}_insertion_link"/>
-      <child link="${prefix}_roll_link"/>
+      <parent link="${prefix}insertion_link"/>
+      <child link="${prefix}roll_link"/>
       <origin rpy="0 0 0" xyz="0 0 0.3829"/>
       <axis xyz="0 0 1"/>
@@ -190,5 +190,5 @@
       <limit effort="100.0" lower="-${PI/2}" upper="${PI/2}" velocity="10"/>
     </joint>
-    <link name="${prefix}_roll_link">
+    <link name="${prefix}roll_link">
       <visual>
         <origin rpy="0 0 ${PI/2}" xyz="0.0 0 -0.3979"/>
