Commit message: add positioning platform for psm

File: dvrk_model/model/PSM.urdf.xacro (robot description, xacro)
@@ -4,5 +4,5 @@
   <xacro:include filename="$(find dvrk_model)/model/psm.urdf.xacro"/>
   <link name="world"/>
-  <xacro:psm_sca
+  <xacro:pp_psm_sca
       prefix="$(arg prefix)"
       parent_link="world"

File: dvrk_model/model/psm.urdf.xacro (robot description, xacro)
@@ -2,4 +2,5 @@
 <robot name="dvrk_psm" xmlns:xacro="http://www.ros.org/wiki/xacro">
   <!-- Macros -->
+  <xacro:include filename="$(find dvrk_model)/model/pp.urdf.xacro"/>
   <xacro:include filename="$(find dvrk_model)/model/psm.base.urdf.xacro"/>
   <xacro:include filename="$(find dvrk_model)/model/psm.tool.sca.urdf.xacro"/>
@@ -11,4 +12,18 @@
         parent_link="${parent_link}"
         xyz="${xyz}" rpy="${rpy}"/>
+    <xacro:psm_tool_sca
+        prefix="${prefix}"/>
+  </xacro:macro>
+  <!-- Macro for psm with sca on a positioning platform -->
+  <xacro:macro name="pp_psm_sca" params="prefix parent_link xyz rpy">
+    <xacro:pp
+	prefix="${prefix}"
+	parent_link="${parent_link}"
+	xyz="${xyz}" rpy="${rpy}"
+	/>
+    <xacro:psm
+        prefix="${prefix}"
+        parent_link="platform"
+        xyz="0 0 0" rpy="0 0 0"/>
     <xacro:psm_tool_sca
         prefix="${prefix}"/>
