Commit message: modify comments in psm.base.urdf.xacro

File: dvrk_model/model/psm.base.urdf.xacro (robot description, xacro)
@@ -2,12 +2,12 @@
 <robot name="dvrk_psm" xmlns:xacro="http://www.ros.org/wiki/xacro">
   <xacro:macro name="psm" params="prefix parent_link xyz rpy">
-    <!-- fixed joint -->
+    <!-- frame 0: base link -->
     <joint name="fixed" type="fixed">
       <parent link="${parent_link}"/>
-      <child link="${prefix}psm_base_link"/>
+      <child link="${prefix}base_link"/>
       <origin rpy="${rpy}" xyz="${xyz}"/>
     </joint>
-    <!-- link 0: psm base link -->
-    <link name="${prefix}psm_base_link">
+    <!-- link 0: base link -->
+    <link name="${prefix}base_link">
       <visual>
         <origin rpy="1.5708 0 3.1416" xyz="0.039 -0.40788 -0.07879"/>
@@ -17,7 +17,7 @@
       </visual>
     </link>
-    <!-- joint 1 -->
+    <!-- frame 1: outer yaw -->
     <joint name="outer_yaw" type="revolute">
-      <parent link="${prefix}psm_base_link"/>
+      <parent link="${prefix}base_link"/>
       <child link="${prefix}outer_yaw_link"/>
       <axis xyz="0 0 1"/>
@@ -26,5 +26,5 @@
       <limit lower="-1.5707" upper="1.5707" velocity=".4" effort="1000"/>
     </joint>
-    <!-- link 1: outer_yaw -->
+    <!-- link 1: outer yaw link -->
     <link name="${prefix}outer_yaw_link">
       <visual>        <!-- <origin rpy="0 0 -1.5708" xyz="0.0125 0 0.1575"/> -->
@@ -38,5 +38,5 @@
     <!-- mechanism, so the outer_pitch_link does not have visual -->
     <!-- link, all visual links mimic outer_pitch value -->
-    <!-- joint 2: outer_pitch -->
+    <!-- frame 2: outer pitch -->
     <joint name="outer_pitch" type="revolute">
       <parent link="${prefix}outer_yaw_link"/>
@@ -46,7 +46,7 @@
       <limit lower="-0.7854" upper="0.7854" velocity=".4" effort="1000"/>
     </joint>
-    <!-- link 2: outer_pitch_link -->
+    <!-- link 2: outer pitch link -->
     <link name="${prefix}outer_pitch_link"/>
-    <!-- joint 2-1: outer_pitch_1 -->
+    <!-- frame 2-1: outer pitch back -->
     <joint name="outer_pitch_1" type="continuous">
       <parent link="${prefix}outer_yaw_link"/>
@@ -57,5 +57,5 @@
       <mimic joint="outer_pitch" multiplier="1"/>
     </joint>
-    <!-- link 2-1: outer_pitch_back -->
+    <!-- link 2-1: outer pitch back link -->
     <link name="${prefix}outer_pitch_back_link">
       <visual>
@@ -66,5 +66,5 @@
       </visual>
     </link>
-    <!-- joint 2-2: outer_pitch_2 -->
+    <!-- frame 2-2: outer pitch front -->
     <joint name="outer_pitch_2" type="continuous">
       <parent link="${prefix}outer_yaw_link"/>
@@ -74,5 +74,5 @@
       <mimic joint="outer_pitch" multiplier="1"/>
     </joint>
-    <!-- link 2-2: outer_pitch_front -->
+    <!-- link 2-2: outer pitch front link -->
     <link name="${prefix}outer_pitch_front_link">
       <visual>
@@ -83,5 +83,5 @@
       </visual>
     </link>
-    <!-- joint 2-3: outer_pitch_3 -->
+    <!-- frame 2-3: outer pitch bottom -->
     <joint name="outer_pitch_3" type="continuous">
       <parent link="${prefix}outer_pitch_back_link"/>
@@ -91,5 +91,5 @@
       <mimic joint="outer_pitch" multiplier="-1"/>
     </joint>
-    <!-- link 2-3: outer_pitch_bottom -->
+    <!-- link 2-3: outer pitch bottom link -->
     <link name="${prefix}outer_pitch_bottom_link">
       <visual>
@@ -100,5 +100,5 @@
       </visual>
     </link>
-    <!-- joint 2-4: outer_pitch_4 -->
+    <!-- frame 2-4: outer pitch top -->
     <joint name="outer_pitch_4" type="continuous">
       <parent link="${prefix}outer_pitch_back_link"/>
@@ -108,5 +108,5 @@
       <mimic joint="outer_pitch" multiplier="-1"/>
     </joint>
-    <!-- link 2-4: outer_pitch_top -->
+    <!-- link 2-4: outer pitch top link -->
     <link name="${prefix}outer_pitch_top_link">
       <visual>
@@ -117,5 +117,5 @@
       </visual>
     </link>
-    <!-- joint 2-5: outer_pitch_5 -->
+    <!-- frame 2-5: outer insertion -->
     <joint name="outer_pitch_5" type="continuous">
       <parent link="${prefix}outer_pitch_bottom_link"/>
@@ -125,5 +125,5 @@
       <mimic joint="outer_pitch" multiplier="1"/>
     </joint>
-    <!-- link 2-5: outer_insertion -->
+    <!-- link 2-5: outer insertion link -->
     <link name="${prefix}outer_insertion_link">
       <visual>
@@ -134,5 +134,5 @@
       </visual>
     </link>
-    <!-- joint 3: insertion -->
+    <!-- frame 3: tool main -->
     <joint name="outer_insertion" type="prismatic">
       <!-- <parent link="${prefix}outer_insertion_link"/> -->
@@ -144,5 +144,5 @@
       <limit lower="0" upper="0.240" velocity=".4" effort="1000"/>
     </joint>
-    <!-- link 3: tool_main_link -->
+    <!-- link 3: tool main link -->
     <link name="${prefix}tool_main_link">
       <visual>
@@ -153,5 +153,5 @@
       </visual>
     </link>
-    <!-- joint 4: Outer Roll -->
+    <!-- frame 4: tool wrist -->
     <joint name="outer_roll" type="revolute">
       <parent link="${prefix}tool_main_link"/>
@@ -161,5 +161,5 @@
       <limit lower="-2.2689" upper="2.2689" velocity=".4" effort="1000"/>
     </joint>
-    <!-- link 4: tool_wrist_link -->
+    <!-- link 4: tool wrist link -->
     <link name="${prefix}tool_wrist_link">
       <visual>
@@ -170,5 +170,5 @@
       </visual>
     </link>
-    <!-- joint 4-1: outer roll shaft joint FIXED-->
+    <!-- frame 4-1: outer roll shaft FIXED-->
     <joint name="outer_roll_shaft" type="fixed">
       <parent link="${prefix}tool_wrist_link"/>
@@ -177,5 +177,5 @@
       <origin rpy="0 0 0" xyz="0 0 0.0"/>
     </joint>
-    <!-- link 4-1: tool_wrist_shaft_link -->
+    <!-- link 4-1: tool wrist shaft link -->
     <link name="${prefix}tool_wrist_shaft_link">
       <visual>
