Commit message: modify limit for the ECM first joint (yaw); add camera frame

File: dvrk_model/model/ecm.urdf.xacro (robot description, xacro)
@@ -48,5 +48,6 @@
       <!--rotates about z axis-->
       <!--limit effort and velocity picked arbitrarily check-->
-      <limit effort="50.0" lower="${-75/180*PI}" upper="${PI/4}" velocity="2"/>
+      <!-- <limit effort="50.0" lower="${-75/180*PI}" upper="${PI/4}" velocity="2"/> -->
+      <limit effort="50.0" lower="${-PI/4}" upper="${PI/4}" velocity="2"/>
       <joint_properties damping="1.0" friction="0.0"/>
     </joint>
@@ -205,4 +206,10 @@
       </collision>
     </link>
+    <joint name="handToCam" type="fixed">
+      <parent link="${prefix}roll_link"/>
+      <child link="${prefix}camera"/>
+      <origin rpy="-0.0129 0.0136 1.5374" xyz="0.000702 -0.0029 0.0036"/>
+    </joint>
+    <link name="${prefix}camera"/>
   </xacro:macro>
 </robot>
